File: board/co2-detector.kicad_pcb (KiCad board)
At the start: 2 copper layers, 37.5 x 51.4 mm, 14 parts, among them U1 WeMos_D1_mini, U2 SGP30

Commit message: Board revision 2, fixes two desing problems
Parts:
- removed the REF** at (139.5, 52.5)
- removed the REF** at (139.5, 93.0)
- removed the REF** at (107.5, 93.0)
- removed the REF** at (107.5, 52.5)
- added REF**: MountingHole_2.2mm_M2, Mounting_Holes:MountingHole_2.2mm_M2, F.Cu at (138.0, 93.2)
- added REF**: MountingHole_2.2mm_M2, Mounting_Holes:MountingHole_2.2mm_M2, F.Cu at (139.4, 52.4)
- added REF**: MountingHole_2.2mm_M2, Mounting_Holes:MountingHole_2.2mm_M2, F.Cu at (107.6, 52.4)
- moved U2 9.14 mm to (131.2, 98.0), turned to 90 degrees
- moved DHT22 3.37 mm to (120.2, 95.6), turned to 0 degrees
- moved R4 2.30 mm to (110.2, 91.8)
- renumbered D3 to G, D1 to R, D2 to Y
Connections:
- U2 pad 3: Net-(U1-Pad14) -> Net-(U1-Pad13)
- U2 pad 4: Net-(U1-Pad13) -> Net-(U1-Pad14)
Routing:
- net /3.3V: track 42.8 -> 53.1 mm
- net /GND: track 95.5 -> 85.9 mm
- net /5V: track 20.9 -> 14.0 mm
- net Net-(U1-Pad14): track 12.5 -> 15.8 mm
- net Net-(U1-Pad13): track 12.5 -> 15.1 mm
- net Net-(R4-Pad2): track 63.6 -> 61.5 mm
Other:
- board text added: "CO2 Detector Rev 2 https://github.com/deuteros76/co2-detector"
- board text removed: "Meteo-home https://github.com/deuteros76/meteo-home"
